Commit message: Fixed typos in many files

File: urdf/materials.xacro (robot description, xacro)
@@ -1,3 +1,4 @@
 <?xml version="1.0"?>
+<!-- Definicion de materiales y colores para Simulación/Visualización -->
 <robot>
   <material name="black">

File: urdf/serial3_robot_v3.xacro (robot description, xacro)
@@ -4,5 +4,5 @@
     <!--Importamos los elementos de personalización de Gazebo -->
     <xacro:include filename="$(find serial3_robot_v3)/urdf/materials.xacro" />
-    <!-- Importamos el archivo de colores para RViz -->
+    <!-- Importamos el archivo de colores para RViz/Gazebo -->
     <xacro:include filename="$(find serial3_robot_v3)/urdf/serial3_robot_v3.gazebo" />
     <!-- Declaramos un "dummy" para fijar 'base_link' en Gazebo -->
@@ -50,5 +50,5 @@
     <link name="e1_link">
         <collision>
-            <origin xyz="0 0 0"rpy="0 0 0" />
+            <origin xyz="0 0 0" rpy="0 0 0" />
             <geometry>
                 <mesh filename="package://serial3_robot_v3/meshes/collision/e1_link.STL" />
