Commit message: Modified xacro file

File: urdf/serial3_robot_v3.xacro (robot description, xacro)
@@ -3,7 +3,7 @@
 <robot name="serial3v3" xmlns:xacro="http://www.ros.org/wiki/xacro">
     <!--Importamos los elementos de personalización de Gazebo -->
-    <xacro:include filename="$(find m2wr_description)/urdf/materials.xacro" />
+    <xacro:include filename="$(find serial3_robot_v3)/urdf/materials.xacro" />
     <!-- Importamos el archivo de colores para RViz -->
-    <xacro:include filename="$(find m2wr_description)/urdf/m2wr.gazebo" />
+    <xacro:include filename="$(find serial3_robot_v3)/urdf/serial3_robot_v3.gazebo" />
     <!-- Declaramos un "dummy" para fijar 'base_link' en Gazebo -->
     <link name="world" />
@@ -37,5 +37,5 @@
                 iyz="1.1648E-12"
                 izz="4.9838E-05" />
-            </inertial>
+        </inertial>
     </link>
     <!-- Definimos a la junta que une al eslabón anterior con el siguiente -->
@@ -176,2 +176,34 @@
         </inertial>
     </link>
+    <!-- Agregamos la Configuración de los motores/actuadores -->
+    <transmission name="trans_base_to_e1_joint">
+        <type>transmission_interface/SimpleTransmission</type>
+        <joint name="base_to_e1_joint">
+            <hardwareInterface>hardware_interface/PositionJointInterface</hardwareInterface>
+        </joint>
+        <actuator name="base_to_e1_joint_motor">
+            <hardwareInterface>hardware_interface/PositionJointInterface</hardwareInterface>
+            <mechanicalReduction>1</mechanicalReduction>
+        </actuator>
+    </transmission>
+    <transmission name="trans_e1_to_e2_joint">
+        <type>transmission_interface/SimpleTransmission</type>
+        <joint name="e1_to_e2_joint">
+            <hardwareInterface>hardware_interface/PositionJointInterface</hardwareInterface>
+        </joint>
+        <actuator name="e1_to_e2_joint_motor">
+            <hardwareInterface>hardware_interface/PositionJointInterface</hardwareInterface>
+            <mechanicalReduction>1</mechanicalReduction>
+        </actuator>
+    </transmission>
+    <transmission name="trans_e2_to_e3_joint">
+        <type>transmission_interface/SimpleTransmission</type>
+        <joint name="e2_to_e3_joint">
+            <hardwareInterface>hardware_interface/PositionJointInterface</hardwareInterface>
+        </joint>
+        <actuator name="e2_to_e3_joint_motor">
+            <hardwareInterface>hardware_interface/PositionJointInterface</hardwareInterface>
+            <mechanicalReduction>1</mechanicalReduction>
+        </actuator>
+    </transmission>
+</robot>

Commit message: Added more xacro files

File: urdf/serial3_robot_v3.xacro (robot description, xacro)
@@ -5,5 +5,7 @@
     <xacro:include filename="$(find serial3_robot_v3)/urdf/materials.xacro" />
     <!-- Importamos el archivo de colores para RViz/Gazebo -->
-    <xacro:include filename="$(find serial3_robot_v3)/urdf/serial3_robot_v3.gazebo.xacro" />
+    <xacro:include filename="$(find serial3_robot_v3)/urdf/serial3v3.gazebo.xacro" />
+     <!-- Importamos el archivo de configuración de transmision para motores -->
+    <xacro:include filename="$(find serial3_robot_v3)/urdf/serial3v3.transmission.xacro" />
     <!-- Declaramos un "dummy" para fijar 'base_link' en Gazebo -->
     <link name="world" />
@@ -176,34 +178,3 @@
         </inertial>
     </link>
-    <!-- Agregamos la Configuración de los motores/actuadores -->
-    <transmission name="trans_base_to_e1_joint">
-        <type>transmission_interface/SimpleTransmission</type>
-        <joint name="base_to_e1_joint">
-            <hardwareInterface>hardware_interface/PositionJointInterface</hardwareInterface>
-        </joint>
-        <actuator name="base_to_e1_joint_motor">
-            <hardwareInterface>hardware_interface/PositionJointInterface</hardwareInterface>
-            <mechanicalReduction>1</mechanicalReduction>
-        </actuator>
-    </transmission>
-    <transmission name="trans_e1_to_e2_joint">
-        <type>transmission_interface/SimpleTransmission</type>
-        <joint name="e1_to_e2_joint">
-            <hardwareInterface>hardware_interface/PositionJointInterface</hardwareInterface>
-        </joint>
-        <actuator name="e1_to_e2_joint_motor">
-            <hardwareInterface>hardware_interface/PositionJointInterface</hardwareInterface>
-            <mechanicalReduction>1</mechanicalReduction>
-        </actuator>
-    </transmission>
-    <transmission name="trans_e2_to_e3_joint">
-        <type>transmission_interface/SimpleTransmission</type>
-        <joint name="e2_to_e3_joint">
-            <hardwareInterface>hardware_interface/PositionJointInterface</hardwareInterface>
-        </joint>
-        <actuator name="e2_to_e3_joint_motor">
-            <hardwareInterface>hardware_interface/PositionJointInterface</hardwareInterface>
-            <mechanicalReduction>1</mechanicalReduction>
-        </actuator>
-    </transmission>
 </robot>

File: urdf/serial3v3.gazebo.xacro (robot description, xacro)
@@ -1,4 +1,7 @@
 <?xml version="1.0"?>
-<robot>
+<robot xmlns:sensor="http://playerstage.sourceforge.net/gazebo/xmlschema/#sensor"
+       xmlns:controller="http://playerstage.sourceforge.net/gazebo/xmlschema/#controller"
+       xmlns:interface="http://playerstage.sourceforge.net/gazebo/xmlschema/#interface"
+       xmlns:xacro="http://ros.org/wiki/xacro">
   <!-- ros_control plugin -->
   <gazebo>
@@ -11,20 +14,25 @@
   <gazebo reference="base_link">
     <material>Gazebo/Grey</material>
+    <turnGravityOff>false</turnGravityOff>
   </gazebo>
   <!-- Link2 -->
   <gazebo reference="e1_link">
     <material>Gazebo/Black</material>
+    <turnGravityOff>false</turnGravityOff>
   </gazebo>
   <!-- Link3 -->
   <gazebo reference="e2_link">
     <material>Gazebo/Black</material>
+    <turnGravityOff>false</turnGravityOff>
   </gazebo>
 <!-- Link4 -->
   <gazebo reference="e3_link">
     <material>Gazebo/Black</material>
+    <turnGravityOff>false</turnGravityOff>
   </gazebo>
  <!-- Link5 -->
   <gazebo reference="end_effector">
     <material>Gazebo/Grey</material>
+    <turnGravityOff>false</turnGravityOff>
   </gazebo>
 </robot>
