Commit message: updated readme and urdf

File: urdf/serial3_robot_v3.xacro (robot description, xacro)
@@ -7,5 +7,5 @@
     <xacro:include filename="$(find serial3_robot_v3)/urdf/serial3v3.gazebo.xacro" />
      <!-- Importamos el archivo de configuración de transmision para motores -->
-    <xacro:include filename="$(find serial3_robot_v3)/urdf/serial3v3.transmission.xacro" />
+    <xacro:include filename="$(find serial3_robot_v3)/urdf/serial3v3_transmission.xacro" />
     <!-- Declaramos un "dummy" para fijar 'base_link' en Gazebo -->
     <link name="world" />
@@ -47,4 +47,5 @@
         <origin xyz="0 0 0.04815" rpy="0 0 0.025007" />
         <axis xyz="0 0 -1" />
+        <limit lower="-1.5708" upper="1.5708" effort="77" velocity="1.43" />
         <dynamics damping="0.7"/>
     </joint>
@@ -81,4 +82,5 @@
         <origin xyz="0 0.00025 0.0305" rpy="1.5708 -1.5679 0" />
         <axis xyz="0 0 -1" />
+        <limit lower="-1.5708" upper="1.5708" effort="133" velocity="1.29" />
         <dynamics damping="0.7"/>
     </joint>
@@ -115,4 +117,5 @@
         <origin xyz="0.237 0 0.00025" rpy="0 0 0.017666" />
         <axis xyz="0 0 -1" />
+        <limit lower="-1.5708" upper="1.5708" effort="66" velocity="2.13" />
         <dynamics damping="0.7"/>
     </joint>
@@ -143,5 +146,5 @@
                 izz="3.9543E-06" />
         </inertial>
-    <link/>
+    </link>
     <joint name="e3_to_end_effector_joint" type="fixed">
         <parent link="e3_link" />

File: urdf/serial3v3_transmission.xacro (robot description, xacro)
@@ -8,8 +8,8 @@
         <type>transmission_interface/SimpleTransmission</type>
         <joint name="base_to_e1_joint">
-            <hardwareInterface>hardware_interface/PositionJointInterface</hardwareInterface>
+            <hardwareInterface>hardware_interface/EffortJointInterface</hardwareInterface>
         </joint>
         <actuator name="base_to_e1_joint_motor">
-            <hardwareInterface>hardware_interface/PositionJointInterface</hardwareInterface>
+            <hardwareInterface>hardware_interface/EffortJointInterface</hardwareInterface>
             <mechanicalReduction>1</mechanicalReduction>
         </actuator>
@@ -18,8 +18,8 @@
         <type>transmission_interface/SimpleTransmission</type>
         <joint name="e1_to_e2_joint">
-            <hardwareInterface>hardware_interface/PositionJointInterface</hardwareInterface>
+            <hardwareInterface>hardware_interface/EffortJointInterface</hardwareInterface>
         </joint>
         <actuator name="e1_to_e2_joint_motor">
-            <hardwareInterface>hardware_interface/PositionJointInterface</hardwareInterface>
+            <hardwareInterface>hardware_interface/EffortJointInterface</hardwareInterface>
             <mechanicalReduction>1</mechanicalReduction>
         </actuator>
@@ -28,8 +28,8 @@
         <type>transmission_interface/SimpleTransmission</type>
         <joint name="e2_to_e3_joint">
-            <hardwareInterface>hardware_interface/PositionJointInterface</hardwareInterface>
+            <hardwareInterface>hardware_interface/EffortJointInterface</hardwareInterface>
         </joint>
         <actuator name="e2_to_e3_joint_motor">
-            <hardwareInterface>hardware_interface/PositionJointInterface</hardwareInterface>
+            <hardwareInterface>hardware_interface/EffortJointInterface</hardwareInterface>
             <mechanicalReduction>1</mechanicalReduction>
         </actuator>
