Commit message: Removed velocity and effort values from URDF

File: urdf/serial3_robot_v3.urdf (robot description, URDF)
Before this commit: robot serial3_robot_v3, 6 links, 5 joints
Joints:
- joint base_to_e1_joint: limit lower=-1.5708 upper=1.5708 effort=77 velocity=1.43117 -> lower=-1.5708 upper=1.5708 effort=0.0 velocity=0.0
- joint e1_to_e2_joint: limit lower=-1.5708 upper=1.5708 effort=133 velocity=1.291543 -> lower=-1.5708 upper=1.5708 effort=0.0 velocity=0.0
- joint e2_to_e3_joint: limit lower=-1.5708 upper=1.5708 effort=66 velocity=2.1293 -> lower=-1.5708 upper=1.5708 effort=0.0 velocity=0.0

Commit message: Added effort and velocity values to URDF

File: urdf/serial3_robot_v3.urdf (robot description, URDF)
Before this commit: robot serial3_robot_v3, 6 links, 5 joints
Joints:
- joint base_to_e1_joint: limit lower=-1.5708 upper=1.5708 effort=0.0 velocity=0.0 -> lower=-1.5708 upper=1.5708 effort=77 velocity=1.43
- joint e1_to_e2_joint: limit lower=-1.5708 upper=1.5708 effort=0.0 velocity=0.0 -> lower=-1.5708 upper=1.5708 effort=133 velocity=1.29
- joint e2_to_e3_joint: limit lower=-1.5708 upper=1.5708 effort=0.0 velocity=0.0 -> lower=-1.5708 upper=1.5708 effort=66 velocity=2.13
